Commit message: Added the mess with proper orientation and inertia values

File: dynaarm_end_effectors/urdf/weight_5kg.urdf.xacro (robot description, xacro)
@@ -27,10 +27,10 @@
     <!-- Inertial Properties -->
     <inertial>
-      <origin xyz="0 0 0" rpy="0 0 0"/>
-      <mass value="0.5"/>
+      <origin xyz="0.026295 0 0.000104" rpy="0 0 0"/>
+      <mass value="5.217999"/>
       <inertia
-        ixx="0.001" ixy="0.0"  ixz="0.0"
-        iyy="0.001" iyz="0.0"
-        izz="0.001"/>
+        ixx="0.031114" ixy="0.0"  ixz="0.000015"
+        iyy="0.015956" iyz="0.0"
+        izz=" 0.019591"/>
     </inertial>
     <!-- Visual -->

Commit message: added collision

File: dynaarm_end_effectors/urdf/weight_5kg.urdf.xacro (robot description, xacro)
@@ -44,11 +44,10 @@
       </material>
     </visual>
-    <!-- Collision
     <collision>
       <origin xyz="0 0 0" rpy="0 0 0"/>
       <geometry>
-        <mesh filename="package://your_package/meshes/end_effector_collision.stl" scale="1 1 1"/>
+      <mesh filename="file://$(find dynaarm_end_effectors)/meshes/weight_mesh.stl" scale="1 1 1"/>
       </geometry>
-    </collision> -->
+    </collision>
   </link>
   <!-- Fixed Joint to parent link -->

Commit message: Adding 200g more to the weight.

File: dynaarm_end_effectors/urdf/weight_5kg.urdf.xacro (robot description, xacro)
@@ -28,5 +28,5 @@
     <inertial>
       <origin xyz="0.026295 0 0.000104" rpy="0 0 0"/>
-      <mass value="5.217999"/>
+      <mass value="5.417999"/>
       <inertia
         ixx="0.031114" ixy="0.0"  ixz="0.000015"
