Commit message: Refactored some params for the URDFs to all have the same names.

File: dynaarm_end_effectors/urdf/freedrive_handle.urdf.xacro (robot description, xacro)
@@ -23,5 +23,5 @@
 <robot name="freedrive_handle" xmlns:xacro="http://www.ros.org/wiki/xacro">
   <!-- Link Definition -->
-<xacro:macro name="freedrive_handle" params="tf_prefix parent_link *origin">
+<xacro:macro name="freedrive_handle" params="tf_prefix parent *origin">
   <link name="${tf_prefix}freedrive_handle_link">
     <!-- Inertial Properties -->
@@ -53,5 +53,5 @@
   <!-- Fixed Joint to parent link -->
   <joint name="${tf_prefix}freedrive_handle_joint" type="fixed">
-    <parent link="${parent_link}"/>
+    <parent link="${parent}"/>
     <child link="${tf_prefix}freedrive_handle_link"/>
     <xacro:insert_block name="origin" />

File: dynaarm_end_effectors/urdf/shovel.urdf.xacro (robot description, xacro)
@@ -23,5 +23,5 @@
 <robot name="shovel" xmlns:xacro="http://www.ros.org/wiki/xacro">
   <!-- Link Definition -->
-<xacro:macro name="shovel" params="tf_prefix parent_link *origin">
+<xacro:macro name="shovel" params="tf_prefix parent *origin">
   <link name="${tf_prefix}shovel_link">
     <!-- Inertial Properties -->
@@ -53,5 +53,5 @@
   <!-- Fixed Joint to parent link -->
   <joint name="${tf_prefix}shovel_joint" type="fixed">
-    <parent link="${parent_link}"/>
+    <parent link="${parent}"/>
     <child link="${tf_prefix}shovel_link"/>
     <xacro:insert_block name="origin" />

File: dynaarm_end_effectors/urdf/shovel_standalone.urdf.xacro (robot description, xacro)
@@ -5,5 +5,5 @@
   <!-- Add platform to world -->
   <xacro:shovel tf_prefix="$(arg tf_prefix)"
-              parent_link="world">
+              parent="world">
     <origin xyz="0 0 0.0" rpy="0 0 0" />
   </xacro:shovel>

File: dynaarm_end_effectors/urdf/weight_5kg.urdf.xacro (robot description, xacro)
@@ -23,5 +23,5 @@
 <robot name="weight_5kg" xmlns:xacro="http://www.ros.org/wiki/xacro">
   <!-- Link Definition -->
-<xacro:macro name="weight_5kg" params="tf_prefix parent_link *origin">
+<xacro:macro name="weight_5kg" params="tf_prefix parent *origin">
   <link name="${tf_prefix}weight_5kg_link">
     <!-- Inertial Properties -->
@@ -53,5 +53,5 @@
   <!-- Fixed Joint to parent link -->
   <joint name="${tf_prefix}weight_5kg_joint" type="fixed">
-    <parent link="${parent_link}"/>
+    <parent link="${parent}"/>
     <child link="${tf_prefix}weight_5kg_link"/>
     <xacro:insert_block name="origin" />

File: dynaarm_end_effectors/urdf/weight_5kg_standalone.urdf.xacro (robot description, xacro)
@@ -5,5 +5,5 @@
   <!-- Add platform to world -->
   <xacro:weight_5kg tf_prefix="$(arg tf_prefix)"
-              parent_link="world">
+              parent="world">
     <origin xyz="0 0 0.0" rpy="0 0 0" />
   </xacro:weight_5kg>
