Commit message: Fixed the mass of the shovel.

File: dynaarm_end_effectors/urdf/shovel.urdf.xacro (robot description, xacro)
@@ -28,5 +28,5 @@
     <inertial>
       <origin xyz="0.004832 -0.001237 0.033429" rpy="0 0 0"/>
-      <mass value="5.417999"/>
+      <mass value="0.551"/>
       <inertia
         ixx="0.001677" ixy="0.0"  ixz="-0.000509"
