Commit message: Added the shovel hook

File: dynaarm_end_effectors/urdf/shovel_gripper.urdf.xacro (robot description, xacro)
@@ -57,4 +57,37 @@
     <xacro:insert_block name="origin" />
   </joint>
+  <link name="${tf_prefix}shovel_hook_link">
+    <!-- Inertial Properties -->
+    <inertial>
+      <origin xyz="0.007887 -0.015220 0.059359" rpy="0 0 0"/>
+      <mass value="0.580724"/>
+      <inertia
+        ixx="0.001822" ixy="0.000232"  ixz="-0.000205"
+        iyy="0.001508" iyz="-0.000158"
+        izz="0.001357"/>
+    </inertial>
+    <!-- Visual -->
+    <visual>
+      <origin xyz="0 0 0" rpy="0 0 0"/>
+      <geometry>
+      <mesh filename="file://$(find dynaarm_end_effectors)/meshes/shovel_hook_mesh.stl" scale="1 1 1"/>
+      </geometry>
+      <material name="gray">
+        <color rgba="0.6 0.6 0.6 1.0"/>
+      </material>
+    </visual>
+    <collision>
+      <origin xyz="0 0 0" rpy="0 0 0"/>
+      <geometry>
+      <mesh filename="file://$(find dynaarm_end_effectors)/meshes/shovel_hook_mesh.stl" scale="1 1 1"/>
+      </geometry>
+    </collision>
+  </link>
+  <!-- Fixed Joint to parent link -->
+  <joint name="${tf_prefix}shovel_hook_joint" type="fixed">
+    <parent link="${tf_prefix}shovel_link"/>
+    <child link="${tf_prefix}shovel_hook_link"/>
+    <xacro:insert_block name="origin" />
+  </joint>
 </xacro:macro>
 </robot>

Commit message: Made the joint revolute

File: dynaarm_end_effectors/urdf/shovel_gripper.urdf.xacro (robot description, xacro)
@@ -84,9 +84,11 @@
     </collision>
   </link>
-  <!-- Fixed Joint to parent link -->
-  <joint name="${tf_prefix}shovel_hook_joint" type="fixed">
+  <!-- Revolute Joint between shovel_link and shovel_hook_link -->
+  <joint name="${tf_prefix}shovel_hook_joint" type="revolute">
     <parent link="${tf_prefix}shovel_link"/>
     <child link="${tf_prefix}shovel_hook_link"/>
-    <xacro:insert_block name="origin" />
+    <origin xyz="0 0 0.05" rpy="0 0 0"/>
+    <axis xyz="0 0 1"/>
+    <limit lower="0" upper="1.57" effort="10" velocity="1"/>
   </joint>
 </xacro:macro>

Commit message: Placed the finger hook properly

File: dynaarm_end_effectors/urdf/shovel_gripper.urdf.xacro (robot description, xacro)
@@ -22,4 +22,5 @@
 -->
 <robot name="shovel_gripper" xmlns:xacro="http://www.ros.org/wiki/xacro">
+<xacro:include filename="$(find dynaarm_description)/urdf/common/dynaarm_common.urdf.xacro" />
   <!-- Link Definition -->
 <xacro:macro name="shovel_gripper" params="tf_prefix parent *origin">
@@ -85,4 +86,5 @@
   </link>
   <!-- Revolute Joint between shovel_link and shovel_hook_link -->
+  <!--
   <joint name="${tf_prefix}shovel_hook_joint" type="revolute">
     <parent link="${tf_prefix}shovel_link"/>
@@ -92,4 +94,16 @@
     <limit lower="0" upper="1.57" effort="10" velocity="1"/>
   </joint>
+  -->
+  <xacro:dynaarm_revolute_joint joint_name="${tf_prefix}shovel_hook_joint"
+    parent="${tf_prefix}shovel_link"
+    child="${tf_prefix}shovel_hook_link"
+    joint_axis_xyz="0 0 1"
+    joint_lower_limit="0"
+    joint_upper_limit="1.57"
+    joint_limit_vel="1"
+    joint_limit_effort="10"
+    joint_type="revolute">
+    <origin xyz="0.0412 -0.0042426 0.053276" rpy="2.3562 0 0" />
+  </xacro:dynaarm_revolute_joint>
 </xacro:macro>
 </robot>
