Commit message: Added the left and right shovel_gripper

File: dynaarm_end_effectors/urdf/shovel_gripper_right.urdf.xacro (robot description, xacro)
@@ -21,7 +21,7 @@
 THE USE OF THIS SOFTWARE, EVEN IF ADVISED OF THE POSSIBILITY OF SUCH DAMAGE.
 -->
-<robot name="shovel_gripper" xmlns:xacro="http://www.ros.org/wiki/xacro">
+<robot name="shovel_gripper_right" xmlns:xacro="http://www.ros.org/wiki/xacro">
   <!-- Link Definition -->
-<xacro:macro name="shovel_gripper" params="tf_prefix parent *origin">
+<xacro:macro name="shovel_gripper_right" params="tf_prefix parent *origin">
   <link name="${tf_prefix}shovel_link">
     <!-- Inertial Properties -->
@@ -38,5 +38,5 @@
       <origin xyz="0 0 0" rpy="0 0 0"/>
       <geometry>
-      <mesh filename="file://$(find dynaarm_end_effectors)/meshes/shovel_gripper_mesh.stl" scale="1 1 1"/>
+      <mesh filename="file://$(find dynaarm_end_effectors)/meshes/shovel_gripper_right_mesh.stl" scale="1 1 1"/>
       </geometry>
       <material name="gray">
@@ -47,5 +47,5 @@
       <origin xyz="0 0 0" rpy="0 0 0"/>
       <geometry>
-      <mesh filename="file://$(find dynaarm_end_effectors)/meshes/shovel_gripper_mesh.stl" scale="1 1 1"/>
+      <mesh filename="file://$(find dynaarm_end_effectors)/meshes/shovel_gripper_right_mesh.stl" scale="1 1 1"/>
       </geometry>
     </collision>
