Commit message: added test for a single dynadrive

File: dynaarm_single_example/dynaarm_single_example_description/urdf/dynaarm_single_example.urdf.xacro (robot description, xacro)
@@ -41,10 +41,6 @@
       </collision>
   </link>
-  <joint name="table_joint" type="fixed">
-        <parent link="world"/>
-        <child link="table"/>
-  </joint>
   <!-- create an instance of the dynaarm xacro macro and fix its base, move it up such that it doesn't intersect with the ground -->
-  <xacro:dynaarm tf_prefix="$(arg tf_prefix)"
+ <!-- <xacro:dynaarm tf_prefix="$(arg tf_prefix)"
                 parent_link="table"
                 dof="$(arg dof)"
@@ -56,4 +52,17 @@
                 version="$(arg version)">
     <origin xyz="0 0 0.085" rpy="0.0 0.0 0.0" />
-  </xacro:dynaarm>
+  </xacro:dynaarm>-->
+    <joint name="test_dynadrive" type="revolute" >
+        <parent link="world"/>
+        <child link="table"/>
+        <limit lower="0.0" upper="1.0" effort="100.0"  velocity="100.0"/>
+  </joint>
+  <xacro:include filename="$(find dynadrive_description)/urdf/dynadrive.ros2control.xacro" />
+  <xacro:dynadrive_ros2_control name="test_dynadrive"
+    ethercat_bus="$(arg ethercat_bus)"
+    start_in_freeze_mode="true"
+    ethercat_address="1"
+    mode="$(arg mode)"
+    >
+  </xacro:dynadrive_ros2_control>
 </robot>
